File: boards/webcam/webcam.kicad_pcb (KiCad board)
At the start: 2 copper layers, 27.5 x 27.5 mm, 48 parts, among them J1 GBCAM, J2 SWD, J3 USBC, J4 SWD, SW1 USB_BOOT, SW2 RESET, U1 RP2040, U2 LMV321, U3 LMV321, U4 W25Q128JVS, U5 XC6206PxxxMR, Y1 X322512MSB4SI

Commit message: pcb: prepare for jlcpcb
Parts:
- J3: footprint Connector_USB:USB_C_Receptacle_HRO_TYPE-C-31-M-12 -> footprints:JLCPCB_USB_C_Receptacle_HRO_TYPE-C-31-M-12
- moved J3 1.44 mm to (43.0, 35.7)
Routing:
- net GND: track 71.7 -> 75.1 mm, vias 19 -> 21
- net +3.3V: track 44.2 -> 40.9 mm, vias 7 -> 5

Commit message: pcb: final prep for jlcpcb
Parts:
- R10, R7, R8, R9: value 51k -> 5.1k
- moved H1 2.94 mm to (32.0, 32.0)
- moved C5 2.36 mm to (34.4, 33.6)
- moved J3 0.10 mm to (43.0, 35.6)
- moved H2 0.10 mm to (55.5, 32.0)
- moved H3 0.10 mm to (55.5, 55.5)
Routing:
- net +3.3V: track 40.9 -> 46.9 mm, vias 5 -> 7
- net /QSPI_SD3: track 20.3 -> 18.8 mm
- net GND: track 75.1 -> 74.9 mm, vias 21 -> 17
Other:
- board text added: "@pimlu"
- board text added: "GBCam"
- board text removed: "Stuart Geipel"
