File: boards/webcam/webcam.kicad_sch (KiCad schematic)
At the start: 48 parts, among them J1 GBCAM, J2 SWD, J3 USBC, J4 SWD, SW1 USB_BOOT, SW2 RESET, U1 RP2040, U2 LMV321, U3 LMV321, U4 W25Q128JVS, U5 XC6206PxxxMR, Y1 X322512MSB4SI

Commit message: pcb: prepare for jlcpcb
Parts:
- R11: now not fitted
Changed lines of the file:
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@@
   )
   (symbol (lib_id "Device:R_Small") (at 149.86 25.4 0) (unit 1)
-    (in_bom yes) (on_board yes) (dnp no)
+    (in_bom yes) (on_board yes) (dnp yes)
     (property "Reference" "R11" (at 151.13 24.13 0)
       (effects (font (size 1.27 1.27)) (justify left))

Commit message: pcb: final prep for jlcpcb
Parts:
- J3: footprint Connector_USB:USB_C_Receptacle_HRO_TYPE-C-31-M-12 -> footprints:JLCPCB_USB_C_Receptacle_HRO_TYPE-C-31-M-12
- R10, R7, R8, R9: value 51k -> 5.1k; LCSC C25794 -> C25905
Changed lines of the file:
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@@
       (effects (font (size 1.27 1.27)) (justify left))
     )
-    (property "Value" "51k" (at 270.51 64.77 0)
+    (property "Value" "5.1k" (at 270.51 64.77 0)
       (effects (font (size 1.27 1.27)) (justify left))
     )
@@
       (effects (font (size 1.27 1.27)) hide)
     )
-    (property "LCSC" "C25794" (at 267.97 63.5 0)
+    (property "LCSC" "C25905" (at 267.97 63.5 0)
       (effects (font (size 1.27 1.27)) hide)
     )
@@
       (effects (font (size 1.27 1.27)) (justify left))
     )
-    (property "Value" "51k" (at 232.41 63.5 0)
+    (property "Value" "5.1k" (at 232.41 63.5 0)
       (effects (font (size 1.27 1.27)) (justify left))
     )
@@
       (effects (font (size 1.27 1.27)) hide)
     )
-    (property "LCSC" "C25794" (at 229.87 62.23 0)
+    (property "LCSC" "C25905" (at 229.87 62.23 0)
       (effects (font (size 1.27 1.27)) hide)
     )
@@
       (effects (font (size 1.27 1.27)) (justify left))
     )
-    (property "Value" "51k" (at 232.41 53.34 0)
+    (property "Value" "5.1k" (at 232.41 53.34 0)
       (effects (font (size 1.27 1.27)) (justify left))
     )
@@
       (effects (font (size 1.27 1.27)) hide)
     )
-    (property "LCSC" "C25794" (at 229.87 52.07 0)
+    (property "LCSC" "C25905" (at 229.87 52.07 0)
       (effects (font (size 1.27 1.27)) hide)
     )
@@
       (effects (font (size 1.27 1.27)))
     )
-    (property "Footprint" "Connector_USB:USB_C_Receptacle_HRO_TYPE-C-31-M-12" (at 34.29 45.72 0)
+    (property "Footprint" "footprints:JLCPCB_USB_C_Receptacle_HRO_TYPE-C-31-M-12" (at 34.29 45.72 0)
       (effects (font (size 1.27 1.27)) hide)
     )
@@
       (effects (font (size 1.27 1.27)) (justify left))
     )
-    (property "Value" "51k" (at 270.51 54.61 0)
+    (property "Value" "5.1k" (at 270.51 54.61 0)
       (effects (font (size 1.27 1.27)) (justify left))
     )
@@
       (effects (font (size 1.27 1.27)) hide)
     )
-    (property "LCSC" "C25794" (at 267.97 53.34 0)
-      (effects (font (size 1.27 1.27)) hide)
-    )
+    (property "LCSC" "C25905" (at 267.97 53.34 0)
+      (effects (font (size 1.27 1.27)) hide)
+    )
